Commit message: Placeholder for thumb dip sensor

File: models/urdf/orcahand.urdf.xacro (robot description, xacro)
@@ -406,4 +406,29 @@
       </collision>
    </link>
+   <link name="${prefix}thumb_dp_sensor_1">
+      <inertial>
+         <origin xyz="0.00233 1e-05 0.01133" rpy="0.00075 0.08211000000000013 0.00013000000000000002"/>
+         <mass value="0.0132"/>
+         <inertia ixx="1.4e-06" iyy="1.37e-06" izz="4.4e-07" ixy="0" ixz="0" iyz="0"/>
+      </inertial>
+      <visual name="${prefix}visual_thumb_dp_1_skin_mesh">
+         <origin xyz="${s * 0.002793435568551968} -6.14386555467744e-07 0.016601042013200628" rpy="3.141592653589793 ${s * -0.40239793279263236} 0.0"/>
+         <geometry>
+            <mesh filename="${rospackage_path}/visual/thumb_dp_1_skin_mesh.stl"
+            scale="${'-1 1 1' if chirality == 'left' else '1 1 1'}"
+            />
+         </geometry>
+         <material name="red"/>
+      </visual>
+      <collision name="${prefix}collision_thumb_dp_1_skin_mesh">
+         <origin xyz="${s * 0.002785448336058668} -6.944475247259374e-06 0.016557497442018437" rpy="3.141592653589793 ${s * -0.3963953079219906} 0.0"/>
+         <geometry>
+            <mesh filename="${rospackage_path}/collision/thumb_dp_1_skin_mesh.stl"
+            scale="${'-1 1 1' if chirality == 'left' else '1 1 1'}"
+            />
+         </geometry>
+         <material name="green"/>
+      </collision>
+   </link>
    <link name="${prefix}thumb_dip_jointbody">
       <inertial>
@@ -425,4 +450,9 @@
       <origin xyz="-0.0 -0.0 -0.0" rpy="0.0 0.0 0.0"/>
    </joint>
+   <joint type="fixed" name="${prefix}thumb_dip_sensor_joint_1">
+      <parent link="${prefix}thumb_dip_jointbody"/>
+      <child link="${prefix}thumb_dp_sensor_1"/>
+      <origin xyz="-0.0 -0.0 -0.0" rpy="0.0 0.0 0.0"/>
+   </joint>
    <link name="${prefix}thumb_fingertip">
       <inertial>
@@ -1160,3 +1190,9 @@
       <color rgba="1 1 1 1"/>
    </material>
+   <material name="red">
+      <color rgba="1 0 0 1"/>
+   </material>
+   <material name="green">
+      <color rgba="0 1 0 1"/>
+   </material>
 </robot>

Commit message: added one thumb contact surface area

File: models/urdf/orcahand.urdf.xacro (robot description, xacro)
@@ -372,5 +372,5 @@
          <origin xyz="${s * 0.001737692119750562} -5.352917438125722e-06 0.005127321105400321" rpy="0.0 ${s * 0.24698289481892632} 0.0"/>
          <geometry>
-            <mesh filename="${rospackage_path}/visual/thumb_dp_mesh.stl"
+            <mesh filename="${rospackage_path}/visual/thumb_dp_mesh_base.stl"
             scale="${'-1 1 1' if chirality == 'left' else '1 1 1'}"
             />
@@ -381,5 +381,5 @@
          <origin xyz="${s * 0.0020244971365026335} 3.68319791392775e-05 0.005533677984084769" rpy="0.24272423187789072 ${s * -0.008190712846545711} ${s * 1.5687682825082248}"/>
          <geometry>
-            <mesh filename="${rospackage_path}/collision/thumb_dp_mesh.stl"
+            <mesh filename="${rospackage_path}/collision/thumb_dp_mesh_base.stl"
             scale="${'-1 1 1' if chirality == 'left' else '1 1 1'}"
             />
@@ -409,11 +409,11 @@
       <inertial>
          <origin xyz="0.00233 1e-05 0.01133" rpy="0.00075 0.08211000000000013 0.00013000000000000002"/>
-         <mass value="0.0132"/>
-         <inertia ixx="1.4e-06" iyy="1.37e-06" izz="4.4e-07" ixy="0" ixz="0" iyz="0"/>
-      </inertial>
-      <visual name="${prefix}visual_thumb_dp_1_skin_mesh">
+         <mass value="1e-8"/>
+         <inertia ixx="1e-8" iyy="1e-8" izz="1e-8" ixy="0.0" ixz="0.0" iyz="0.0"/>
+      </inertial>
+      <visual name="${prefix}visual_thumb_dp_skin_mesh_surface_1">
          <origin xyz="${s * 0.002793435568551968} -6.14386555467744e-07 0.016601042013200628" rpy="3.141592653589793 ${s * -0.40239793279263236} 0.0"/>
          <geometry>
-            <mesh filename="${rospackage_path}/visual/thumb_dp_1_skin_mesh.stl"
+            <mesh filename="${rospackage_path}/visual/thumb_dp_skin_mesh_surface_1.stl"
             scale="${'-1 1 1' if chirality == 'left' else '1 1 1'}"
             />
@@ -421,8 +421,8 @@
          <material name="red"/>
       </visual>
-      <collision name="${prefix}collision_thumb_dp_1_skin_mesh">
+      <collision name="${prefix}collision_thumb_dp_skin_mesh_surface_1">
          <origin xyz="${s * 0.002785448336058668} -6.944475247259374e-06 0.016557497442018437" rpy="3.141592653589793 ${s * -0.3963953079219906} 0.0"/>
          <geometry>
-            <mesh filename="${rospackage_path}/collision/thumb_dp_1_skin_mesh.stl"
+            <mesh filename="${rospackage_path}/collision/thumb_dp_skin_mesh_surface_1.stl"
             scale="${'-1 1 1' if chirality == 'left' else '1 1 1'}"
             />
@@ -448,4 +448,9 @@
       <parent link="${prefix}thumb_dip_jointbody"/>
       <child link="${prefix}thumb_dp"/>
+      <origin xyz="-0.0 -0.0 -0.0" rpy="0.0 0.0 0.0"/>
+   </joint>
+   <joint type="fixed" name="${prefix}thumb_dip_sensor_1_joint">
+      <parent link="${prefix}thumb_dip_jointbody"/>
+      <child link="${prefix}thumb_dp_sensor_1"/>
       <origin xyz="-0.0 -0.0 -0.0" rpy="0.0 0.0 0.0"/>
    </joint>

Commit message: small naming fixes for correct thumb 1

File: models/urdf/orcahand.urdf.xacro (robot description, xacro)
@@ -372,5 +372,5 @@
          <origin xyz="${s * 0.001737692119750562} -5.352917438125722e-06 0.005127321105400321" rpy="0.0 ${s * 0.24698289481892632} 0.0"/>
          <geometry>
-            <mesh filename="${rospackage_path}/visual/thumb_dp_mesh_base.stl"
+            <mesh filename="${rospackage_path}/visual/thumb_dp_mesh.stl"
             scale="${'-1 1 1' if chirality == 'left' else '1 1 1'}"
             />
@@ -381,5 +381,5 @@
          <origin xyz="${s * 0.0020244971365026335} 3.68319791392775e-05 0.005533677984084769" rpy="0.24272423187789072 ${s * -0.008190712846545711} ${s * 1.5687682825082248}"/>
          <geometry>
-            <mesh filename="${rospackage_path}/collision/thumb_dp_mesh_base.stl"
+            <mesh filename="${rospackage_path}/collision/thumb_dp_mesh.stl"
             scale="${'-1 1 1' if chirality == 'left' else '1 1 1'}"
             />
@@ -390,5 +390,5 @@
          <origin xyz="${s * 0.002793435568551968} -6.14386555467744e-07 0.016601042013200628" rpy="3.141592653589793 ${s * -0.40239793279263236} 0.0"/>
          <geometry>
-            <mesh filename="${rospackage_path}/visual/thumb_dp_skin_mesh.stl"
+            <mesh filename="${rospackage_path}/visual/thumb_dp_skin_mesh_base.stl"
             scale="${'-1 1 1' if chirality == 'left' else '1 1 1'}"
             />
@@ -399,5 +399,5 @@
          <origin xyz="${s * 0.002785448336058668} -6.944475247259374e-06 0.016557497442018437" rpy="3.141592653589793 ${s * -0.3963953079219906} 0.0"/>
          <geometry>
-            <mesh filename="${rospackage_path}/collision/thumb_dp_skin_mesh.stl"
+            <mesh filename="${rospackage_path}/collision/thumb_dp_skin_mesh_base.stl"
             scale="${'-1 1 1' if chirality == 'left' else '1 1 1'}"
             />
@@ -451,9 +451,4 @@
    </joint>
    <joint type="fixed" name="${prefix}thumb_dip_sensor_1_joint">
-      <parent link="${prefix}thumb_dip_jointbody"/>
-      <child link="${prefix}thumb_dp_sensor_1"/>
-      <origin xyz="-0.0 -0.0 -0.0" rpy="0.0 0.0 0.0"/>
-   </joint>
-   <joint type="fixed" name="${prefix}thumb_dip_sensor_joint_1">
       <parent link="${prefix}thumb_dip_jointbody"/>
       <child link="${prefix}thumb_dp_sensor_1"/>
