Commit message: correct chirality && prefix

File: models/urdf/orcahand.urdf (robot description, URDF)
Before this commit: robot orcahand, 43 links, 42 joints
Links:
- removed link myprefix_index_abd_jointbody
- removed link myprefix_index_fingertip
- removed link myprefix_index_ip
- removed link myprefix_index_mcp_jointbody
- removed link myprefix_index_mp
- removed link myprefix_index_pip_jointbody
- removed link myprefix_index_pp
- removed link myprefix_middle_abd_jointbody
- removed link myprefix_middle_fingertip
- removed link myprefix_middle_ip
- removed link myprefix_middle_mcp_jointbody
- removed link myprefix_middle_mp
- removed link myprefix_middle_pip_jointbody
- removed link myprefix_middle_pp
- removed link myprefix_palm
- removed link myprefix_pinky_abd_jointbody
- removed link myprefix_pinky_fingertip
- removed link myprefix_pinky_ip
- removed link myprefix_pinky_mcp_jointbody
- removed link myprefix_pinky_mp
- removed link myprefix_pinky_pip_jointbody
- removed link myprefix_pinky_pp
- removed link myprefix_ring_abd_jointbody
- removed link myprefix_ring_fingertip
- removed link myprefix_ring_ip
- removed link myprefix_ring_mcp_jointbody
- removed link myprefix_ring_mp
- removed link myprefix_ring_pip_jointbody
- removed link myprefix_ring_pp
- removed link myprefix_root
- removed link myprefix_thumb_abd_jointbody
- removed link myprefix_thumb_dip_jointbody
- removed link myprefix_thumb_dp
- removed link myprefix_thumb_dp_sensor_1
- removed link myprefix_thumb_fingertip
- removed link myprefix_thumb_ip
- removed link myprefix_thumb_mcp_jointbody
- removed link myprefix_thumb_mp
- removed link myprefix_thumb_pip_jointbody
- removed link myprefix_thumb_pp
- removed link myprefix_tower
- removed link myprefix_world2tower_fixed_jointbody
- removed link myprefix_wrist_jointbody
- added link right_index_abd_jointbody, mass 0.001
- added link right_index_fingertip, mass 0.0
- added link right_index_ip, mass 0.01521; collision mesh filename=package://orcahand_description/assets/urdf/collision/index_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 scale=1 1 1; collision mesh filename=package://orcahand_description/assets/urdf/collision/index_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 scale=1 1 1
- added link right_index_mcp_jointbody, mass 0.001
- added link right_index_mp, mass 0.00498; collision mesh filename=package://orcahand_description/assets/urdf/collision/index_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 scale=1 1 1; visual mesh filename=package://orcahand_description/assets/urdf/visual/index_mp_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 scale=1 1 1
- added link right_index_pip_jointbody, mass 0.001
- added link right_index_pp, mass 0.0165; collision mesh filename=package://orcahand_description/assets/urdf/collision/index_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 scale=1 1 1; collision mesh filename=package://orcahand_description/assets/urdf/collision/index_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 scale=1 1 1
- added link right_middle_abd_jointbody, mass 0.001
- added link right_middle_fingertip, mass 0.0
- added link right_middle_ip, mass 0.01521; collision mesh filename=package://orcahand_description/assets/urdf/collision/middle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 scale=1 1 1; collision mesh filename=package://orcahand_description/assets/urdf/collision/middle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 scale=1 1 1
- added link right_middle_mcp_jointbody, mass 0.001
- added link right_middle_mp, mass 0.00498; collision mesh filename=package://orcahand_description/assets/urdf/collision/middle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 scale=1 1 1; visual mesh filename=package://orcahand_description/assets/urdf/visual/middle_mp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 scale=1 1 1
- added link right_middle_pip_jointbody, mass 0.001
- added link right_middle_pp, mass 0.02006; collision mesh filename=package://orcahand_description/assets/urdf/collision/middle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 scale=1 1 1; collision mesh filename=package://orcahand_description/assets/urdf/collision/middle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 scale=1 1 1
- added link right_palm, mass 0.0257; collision mesh filename=package://orcahand_description/assets/urdf/collision/palm_m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 scale=1 1 1; collision mesh filename=package://orcahand_description/assets/urdf/collision/palm_s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 scale=1 1 1
- added link right_pinky_abd_jointbody, mass 0.001
- added link right_pinky_fingertip, mass 0.0
- added link right_pinky_ip, mass 0.01521; collision mesh filename=package://orcahand_description/assets/urdf/collision/pinky_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 scale=1 1 1; collision mesh filename=package://orcahand_description/assets/urdf/collision/pinky_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 scale=1 1 1
- added link right_pinky_mcp_jointbody, mass 0.001
- added link right_pinky_mp, mass 0.00498; collision mesh filename=package://orcahand_description/assets/urdf/collision/pinky_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 scale=1 1 1; visual mesh filename=package://orcahand_description/assets/urdf/visual/pinky_mp_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 scale=1 1 1
- added link right_pinky_pip_jointbody, mass 0.001
- added link right_pinky_pp, mass 0.01402; collision mesh filename=package://orcahand_description/assets/urdf/collision/pinky_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 scale=1 1 1; collision mesh filename=package://orcahand_description/assets/urdf/collision/pinky_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 scale=1 1 1
- added link right_ring_abd_jointbody, mass 0.001
- added link right_ring_fingertip, mass 0.0
- added link right_ring_ip, mass 0.01521; collision mesh filename=package://orcahand_description/assets/urdf/collision/ring_i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 scale=1 1 1; collision mesh filename=package://orcahand_description/assets/urdf/collision/ring_i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 scale=1 1 1
- added link right_ring_mcp_jointbody, mass 0.001
- added link right_ring_mp, mass 0.00498; collision mesh filename=package://orcahand_description/assets/urdf/collision/ring_m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 scale=1 1 1; visual mesh filename=package://orcahand_description/assets/urdf/visual/ring_mp_m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 scale=1 1 1
- added link right_ring_pip_jointbody, mass 0.001
- added link right_ring_pp, mass 0.02006; collision mesh filename=package://orcahand_description/assets/urdf/collision/ring_p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 scale=1 1 1; collision mesh filename=package://orcahand_description/assets/urdf/collision/ring_p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 scale=1 1 1
- added link right_root, mass 0.0
- added link right_thumb_abd_jointbody, mass 0.001
- added link right_thumb_dip_jointbody, mass 0.001
- added link right_thumb_dp, mass 0.0132; collision mesh filename=package://orcahand_description/assets/urdf/collision/thumb_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 scale=1 1 1; collision mesh filename=package://orcahand_description/assets/urdf/collision/thumb_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 scale=1 1 1
- added link right_thumb_dp_sensor_1, mass 1e-8; collision mesh filename=package://orcahand_description/assets/urdf/collision/thumb_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 scale=1 1 1; visual mesh filename=package://orcahand_description/assets/urdf/visual/thumb_dp_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 scale=1 1 1
- added link right_thumb_fingertip, mass 0.0
- added link right_thumb_ip, mass 0.01402; collision mesh filename=package://orcahand_description/assets/urdf/collision/thumb_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 scale=1 1 1; collision mesh filename=package://orcahand_description/assets/urdf/collision/thumb_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 scale=1 1 1
- added link right_thumb_mcp_jointbody, mass 0.001
- added link right_thumb_mp, mass 0.00586; collision mesh filename=package://orcahand_description/assets/urdf/collision/thumb_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 scale=1 1 1; visual mesh filename=package://orcahand_description/assets/urdf/visual/thumb_mp_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 scale=1 1 1
- added link right_thumb_pip_jointbody, mass 0.001
- added link right_thumb_pp, mass 0.00655; collision mesh filename=package://orcahand_description/assets/urdf/collision/thumb_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 scale=1 1 1; visual mesh filename=package://orcahand_description/assets/urdf/visual/thumb_pp_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 scale=1 1 1
- added link right_tower, mass 0.9; collision mesh filename=package://orcahand_description/assets/urdf/collision/tower_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 scale=1 1 1; collision mesh filename=package://orcahand_description/assets/urdf/collision/tower_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 scale=1 1 1
- added link right_world2tower_fixed_jointbody, mass 0.001
- added link right_wrist_jointbody, mass 0.001
Joints:
- removed joint myprefix_index_abd
- removed joint myprefix_index_abd_offset
- removed joint myprefix_index_ip2index_fingertip_fixed_offset
- removed joint myprefix_index_mcp
- removed joint myprefix_index_mcp_offset
- removed joint myprefix_index_pip
- removed joint myprefix_index_pip_offset
- removed joint myprefix_middle_abd
- removed joint myprefix_middle_abd_offset
- removed joint myprefix_middle_ip2middle_fingertip_fixed_offset
- removed joint myprefix_middle_mcp
- removed joint myprefix_middle_mcp_offset
- removed joint myprefix_middle_pip
- removed joint myprefix_middle_pip_offset
- removed joint myprefix_pinky_abd
- removed joint myprefix_pinky_abd_offset
- removed joint myprefix_pinky_ip2pinky_fingertip_fixed_offset
- removed joint myprefix_pinky_mcp
- removed joint myprefix_pinky_mcp_offset
- removed joint myprefix_pinky_pip
- removed joint myprefix_pinky_pip_offset
- removed joint myprefix_ring_abd
- removed joint myprefix_ring_abd_offset
- removed joint myprefix_ring_ip2ring_fingertip_fixed_offset
- removed joint myprefix_ring_mcp
- removed joint myprefix_ring_mcp_offset
- removed joint myprefix_ring_pip
- removed joint myprefix_ring_pip_offset
- removed joint myprefix_thumb_abd
- removed joint myprefix_thumb_abd_offset
- removed joint myprefix_thumb_dip
- removed joint myprefix_thumb_dip_offset
- removed joint myprefix_thumb_dip_sensor_1_joint
- removed joint myprefix_thumb_dp2thumb_fingertip_fixed_offset
- removed joint myprefix_thumb_mcp
- removed joint myprefix_thumb_mcp_offset
- removed joint myprefix_thumb_pip
- removed joint myprefix_thumb_pip_offset
- removed joint myprefix_world2tower_fixed
- removed joint myprefix_world2tower_fixed_offset
- removed joint myprefix_wrist
- removed joint myprefix_wrist_offset
- added joint right_index_abd: type revolute, parent right_palm, child right_index_abd_jointbody, origin xyz=-0.024088797002689358 0.0018999642829399502 0.025164928786148736 rpy=1.6066999999999996 1.13552 -0.05339000000000049, axis 0.0 0.0 -1.0, limit lower=-0.645772 upper=0.645772 effort=100 velocity=100
- added joint right_index_abd_offset: type fixed, parent right_index_abd_jointbody, child right_index_mp, origin xyz=-0.02 -0.0 -0.0 rpy=0.0 0.0 0.0
- added joint right_index_ip2index_fingertip_fixed_offset: type fixed, parent right_index_ip, child right_index_fingertip, origin xyz=-0.009 0.0 0.035 rpy=0.0 0.0 0.0
- added joint right_index_mcp: type revolute, parent right_index_mp, child right_index_mcp_jointbody, origin xyz=0.0 0.0 0.0 rpy=3.141592653589793 -1.5707926535897931 3.141592653589793, axis 0.0 -1.0 0.0, limit lower=-0.349066 upper=1.658063 effort=100 velocity=100
- added joint right_index_mcp_offset: type fixed, parent right_index_mcp_jointbody, child right_index_pp, origin xyz=-0.0 -0.0 -0.0 rpy=0.0 0.0 0.0
- added joint right_index_pip: type revolute, parent right_index_pp, child right_index_pip_jointbody, origin xyz=0.0005 0.0 0.038 rpy=0.0 0.0 0.0, axis 0.0 -1.0 0.0, limit lower=-0.349066 upper=1.884956 effort=100 velocity=100
- added joint right_index_pip_offset: type fixed, parent right_index_pip_jointbody, child right_index_ip, origin xyz=-0.0 -0.0 -0.0 rpy=0.0 0.0 0.0
- added joint right_middle_abd: type revolute, parent right_palm, child right_middle_abd_jointbody, origin xyz=-7.346410206776621e-08 0.0 0.030000000000134926 rpy=-1.5707926536208807 1.5707926535897934 3.141592653558706, axis 0.0 0.0 -1.0, limit lower=-0.645772 upper=0.645772 effort=100 velocity=100
- added joint right_middle_abd_offset: type fixed, parent right_middle_abd_jointbody, child right_middle_mp, origin xyz=-0.02 -0.0 -0.0 rpy=0.0 0.0 0.0
- added joint right_middle_ip2middle_fingertip_fixed_offset: type fixed, parent right_middle_ip, child right_middle_fingertip, origin xyz=-0.009 0.0 0.035 rpy=0.0 0.0 0.0
- added joint right_middle_mcp: type revolute, parent right_middle_mp, child right_middle_mcp_jointbody, origin xyz=0.0 0.0 0.0 rpy=3.141592653589793 -1.5707926535897931 3.141592653589793, axis 0.0 -1.0 0.0, limit lower=-0.349066 upper=1.588250 effort=100 velocity=100
- added joint right_middle_mcp_offset: type fixed, parent right_middle_mcp_jointbody, child right_middle_pp, origin xyz=-0.0 -0.0 -0.0 rpy=0.0 0.0 0.0
- added joint right_middle_pip: type revolute, parent right_middle_pp, child right_middle_pip_jointbody, origin xyz=0.0005 0.0 0.046 rpy=0.0 0.0 0.0, axis 0.0 -1.0 0.0, limit lower=-0.349066 upper=1.867502 effort=100 velocity=100
- added joint right_middle_pip_offset: type fixed, parent right_middle_pip_jointbody, child right_middle_ip, origin xyz=-0.0 -0.0 -0.0 rpy=0.0 0.0 0.0
- added joint right_pinky_abd: type revolute, parent right_palm, child right_pinky_abd_jointbody, origin xyz=0.04258452932438962 0.004988143142003794 0.007243722937596895 rpy=-1.49694 0.8614899999999999 -2.8837299999999995, axis 0.0 0.0 -1.0, limit lower=-0.645772 upper=0.645772 effort=100 velocity=100
- added joint right_pinky_abd_offset: type fixed, parent right_pinky_abd_jointbody, child right_pinky_mp, origin xyz=-0.02 -0.0 -0.0 rpy=0.0 0.0 0.0
- added joint right_pinky_ip2pinky_fingertip_fixed_offset: type fixed, parent right_pinky_ip, child right_pinky_fingertip, origin xyz=-0.009 0.0 0.035 rpy=0.0 0.0 0.0
- added joint right_pinky_mcp: type revolute, parent right_pinky_mp, child right_pinky_mcp_jointbody, origin xyz=0.0 0.0 0.0 rpy=3.141592653589793 -1.5707926535897931 3.141592653589793, axis 0.0 -1.0 0.0, limit lower=-0.349066 upper=1.710423 effort=100 velocity=100
- added joint right_pinky_mcp_offset: type fixed, parent right_pinky_mcp_jointbody, child right_pinky_pp, origin xyz=-0.0 -0.0 -0.0 rpy=0.0 0.0 0.0
- added joint right_pinky_pip: type revolute, parent right_pinky_pp, child right_pinky_pip_jointbody, origin xyz=0.0005 0.0 0.033 rpy=0.0 0.0 0.0, axis 0.0 -1.0 0.0, limit lower=-0.349066 upper=1.884956 effort=100 velocity=100
- added joint right_pinky_pip_offset: type fixed, parent right_pinky_pip_jointbody, child right_pinky_ip, origin xyz=-0.0 -0.0 -0.0 rpy=0.0 0.0 0.0
- added joint right_ring_abd: type revolute, parent right_palm, child right_ring_abd_jointbody, origin xyz=0.021521022061295733 0.0015382095479525787 0.020824784431525818 rpy=-1.5359699999999998 1.30836 -3.05441, axis 0.0 0.0 -1.0, limit lower=-0.645772 upper=0.645772 effort=100 velocity=100
- added joint right_ring_abd_offset: type fixed, parent right_ring_abd_jointbody, child right_ring_mp, origin xyz=-0.02 -0.0 -0.0 rpy=0.0 0.0 0.0
- added joint right_ring_ip2ring_fingertip_fixed_offset: type fixed, parent right_ring_ip, child right_ring_fingertip, origin xyz=-0.009 0.0 0.035 rpy=0.0 0.0 0.0
- added joint right_ring_mcp: type revolute, parent right_ring_mp, child right_ring_mcp_jointbody, origin xyz=0.0 0.0 0.0 rpy=3.141592653589793 -1.5707926535897931 3.141592653589793, axis 0.0 -1.0 0.0, limit lower=-0.349066 upper=1.588250 effort=100 velocity=100
- added joint right_ring_mcp_offset: type fixed, parent right_ring_mcp_jointbody, child right_ring_pp, origin xyz=-0.0 -0.0 -0.0 rpy=0.0 0.0 0.0
- added joint right_ring_pip: type revolute, parent right_ring_pp, child right_ring_pip_jointbody, origin xyz=0.0005 0.0 0.046 rpy=0.0 0.0 0.0, axis 0.0 -1.0 0.0, limit lower=-0.349066 upper=1.867502 effort=100 velocity=100
- added joint right_ring_pip_offset: type fixed, parent right_ring_pip_jointbody, child right_ring_ip, origin xyz=-0.0 -0.0 -0.0 rpy=0.0 0.0 0.0
- added joint right_thumb_abd: type revolute, parent right_thumb_mp, child right_thumb_abd_jointbody, origin xyz=6.938893903907228e-18 0.0 0.0 rpy=-1.22173 0.0 0.0, axis 0.0 0.34202085907197166 0.9396923602752502, limit lower=-0.349066 upper=0.733038 effort=100 velocity=100
- added joint right_thumb_abd_offset: type fixed, parent right_thumb_abd_jointbody, child right_thumb_pp, origin xyz=-0.03 -0.0 -0.0 rpy=0.0 0.0 0.0
- added joint right_thumb_dip: type revolute, parent right_thumb_ip, child right_thumb_dip_jointbody, origin xyz=0.0005 0.0 0.033 rpy=0.0 0.0 0.0, axis 0.0 -1.0 0.0, limit lower=-0.349066 upper=1.954769 effort=100 velocity=100
- added joint right_thumb_dip_offset: type fixed, parent right_thumb_dip_jointbody, child right_thumb_dp, origin xyz=-0.0 -0.0 -0.0 rpy=0.0 0.0 0.0
- added joint right_thumb_dip_sensor_1_joint: type fixed, parent right_thumb_dip_jointbody, child right_thumb_dp_sensor_1, origin xyz=-0.0 -0.0 -0.0 rpy=0.0 0.0 0.0
- added joint right_thumb_dp2thumb_fingertip_fixed_offset: type fixed, parent right_thumb_dp, child right_thumb_fingertip, origin xyz=-0.003 0.0 0.025 rpy=0.0 0.0 0.0
- added joint right_thumb_mcp: type revolute, parent right_palm, child right_thumb_mcp_jointbody, origin xyz=-0.02821 0.01777 -0.01321 rpy=0.5385700000000002 -0.05594999999999972 -1.27047, axis 0.0 0.0 -1.0, limit lower=-0.87266 upper=0.87266 effort=100 velocity=100
- added joint right_thumb_mcp_offset: type fixed, parent right_thumb_mcp_jointbody, child right_thumb_mp, origin xyz=-0.0 -0.0 -0.0 rpy=0.0 0.0 0.0
- added joint right_thumb_pip: type revolute, parent right_thumb_pp, child right_thumb_pip_jointbody, origin xyz=0.0 0.0 0.0 rpy=-2.6535897934554242e-06 1.5707926535897934 3.141592653589793, axis 0.0 -1.0 0.0, limit lower=-0.209440 upper=1.884956 effort=100 velocity=100
- added joint right_thumb_pip_offset: type fixed, parent right_thumb_pip_jointbody, child right_thumb_ip, origin xyz=-0.0 -0.0 -0.0 rpy=0.0 0.0 0.0
- added joint right_world2tower_fixed: type fixed, parent right_root, child right_world2tower_fixed_jointbody, origin xyz=-0.04 0.0 0.04575 rpy=0.0 0.0 0.0
- added joint right_world2tower_fixed_offset: type fixed, parent right_world2tower_fixed_jointbody, child right_tower, origin xyz=-0.0 -0.0 -0.0 rpy=0.0 0.0 0.0
- added joint right_wrist: type revolute, parent right_tower, child right_wrist_jointbody, origin xyz=0.04063 0.0 0.10486999999999999 rpy=0.0 0.0 0.0, axis 1.0 0.0 0.0, limit lower=-0.872665 upper=0.523599 effort=100 velocity=100
- added joint right_wrist_offset: type fixed, parent right_wrist_jointbody, child right_palm, origin xyz=-0.002 0.00144 0.03872 rpy=0.0 0.0 0.0
