Commit message: added middle finger contact surfaces

File: models/urdf/orcahand.urdf (robot description, URDF)
Before this commit: robot orcahand, 43 links, 42 joints
Links:
- added link right_middle_ip_sensor_1, mass 1e-8; collision mesh filename=package://orcahand_description/assets/urdf/collision/middle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 scale=1 1 1; visual mesh filename=package://orcahand_description/assets/urdf/visual/middle_ip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 scale=1 1 1
- added link right_middle_ip_sensor_10, mass 1e-8; collision mesh filename=package://orcahand_description/assets/urdf/collision/middle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 scale=1 1 1; visual mesh filename=package://orcahand_description/assets/urdf/visual/middle_ip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 scale=1 1 1
- added link right_middle_ip_sensor_11, mass 1e-8; collision mesh filename=package://orcahand_description/assets/urdf/collision/middle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 scale=1 1 1; visual mesh filename=package://orcahand_description/assets/urdf/visual/middle_ip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 scale=1 1 1
- added link right_middle_ip_sensor_12, mass 1e-8; collision mesh filename=package://orcahand_description/assets/urdf/collision/middle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 scale=1 1 1; visual mesh filename=package://orcahand_description/assets/urdf/visual/middle_ip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 scale=1 1 1
- added link right_middle_ip_sensor_13, mass 1e-8; collision mesh filename=package://orcahand_description/assets/urdf/collision/middle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 scale=1 1 1; visual mesh filename=package://orcahand_description/assets/urdf/visual/middle_ip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 scale=1 1 1
- added link right_middle_ip_sensor_14, mass 1e-8; collision mesh filename=package://orcahand_description/assets/urdf/collision/middle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 scale=1 1 1; visual mesh filename=package://orcahand_description/assets/urdf/visual/middle_ip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 scale=1 1 1
- added link right_middle_ip_sensor_2, mass 1e-8; collision mesh filename=package://orcahand_description/assets/urdf/collision/middle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 scale=1 1 1; visual mesh filename=package://orcahand_description/assets/urdf/visual/middle_ip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 scale=1 1 1
- added link right_middle_ip_sensor_3, mass 1e-8; collision mesh filename=package://orcahand_description/assets/urdf/collision/middle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 scale=1 1 1; visual mesh filename=package://orcahand_description/assets/urdf/visual/middle_ip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 scale=1 1 1
- added link right_middle_ip_sensor_4, mass 1e-8; collision mesh filename=package://orcahand_description/assets/urdf/collision/middle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 scale=1 1 1; visual mesh filename=package://orcahand_description/assets/urdf/visual/middle_ip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 scale=1 1 1
- added link right_middle_ip_sensor_5, mass 1e-8; collision mesh filename=package://orcahand_description/assets/urdf/collision/middle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 scale=1 1 1; visual mesh filename=package://orcahand_description/assets/urdf/visual/middle_ip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 scale=1 1 1
- added link right_middle_ip_sensor_6, mass 1e-8; collision mesh filename=package://orcahand_description/assets/urdf/collision/middle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 scale=1 1 1; visual mesh filename=package://orcahand_description/assets/urdf/visual/middle_ip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 scale=1 1 1
- added link right_middle_ip_sensor_7, mass 1e-8; collision mesh filename=package://orcahand_description/assets/urdf/collision/middle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 scale=1 1 1; visual mesh filename=package://orcahand_description/assets/urdf/visual/middle_ip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 scale=1 1 1
- added link right_middle_ip_sensor_8, mass 1e-8; collision mesh filename=package://orcahand_description/assets/urdf/collision/middle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 scale=1 1 1; visual mesh filename=package://orcahand_description/assets/urdf/visual/middle_ip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 scale=1 1 1
- added link right_middle_ip_sensor_9, mass 1e-8; collision mesh filename=package://orcahand_description/assets/urdf/collision/middle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 scale=1 1 1; visual mesh filename=package://orcahand_description/assets/urdf/visual/middle_ip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 scale=1 1 1
Joints:
- added joint right_middle_pip_sensor_10_joint: type fixed, parent right_middle_pip_jointbody, child right_middle_ip_sensor_10, origin xyz=-0.0 -0.0 -0.0 rpy=0.0 0.0 0.0
- added joint right_middle_pip_sensor_11_joint: type fixed, parent right_middle_pip_jointbody, child right_middle_ip_sensor_11, origin xyz=-0.0 -0.0 -0.0 rpy=0.0 0.0 0.0
- added joint right_middle_pip_sensor_12_joint: type fixed, parent right_middle_pip_jointbody, child right_middle_ip_sensor_12, origin xyz=-0.0 -0.0 -0.0 rpy=0.0 0.0 0.0
- added joint right_middle_pip_sensor_13_joint: type fixed, parent right_middle_pip_jointbody, child right_middle_ip_sensor_13, origin xyz=-0.0 -0.0 -0.0 rpy=0.0 0.0 0.0
- added joint right_middle_pip_sensor_14_joint: type fixed, parent right_middle_pip_jointbody, child right_middle_ip_sensor_14, origin xyz=-0.0 -0.0 -0.0 rpy=0.0 0.0 0.0
- added joint right_middle_pip_sensor_1_joint: type fixed, parent right_middle_pip_jointbody, child right_middle_ip_sensor_1, origin xyz=-0.0 -0.0 -0.0 rpy=0.0 0.0 0.0
- added joint right_middle_pip_sensor_2_joint: type fixed, parent right_middle_pip_jointbody, child right_middle_ip_sensor_2, origin xyz=-0.0 -0.0 -0.0 rpy=0.0 0.0 0.0
- added joint right_middle_pip_sensor_3_joint: type fixed, parent right_middle_pip_jointbody, child right_middle_ip_sensor_3, origin xyz=-0.0 -0.0 -0.0 rpy=0.0 0.0 0.0
- added joint right_middle_pip_sensor_4_joint: type fixed, parent right_middle_pip_jointbody, child right_middle_ip_sensor_4, origin xyz=-0.0 -0.0 -0.0 rpy=0.0 0.0 0.0
- added joint right_middle_pip_sensor_5_joint: type fixed, parent right_middle_pip_jointbody, child right_middle_ip_sensor_5, origin xyz=-0.0 -0.0 -0.0 rpy=0.0 0.0 0.0
- added joint right_middle_pip_sensor_6_joint: type fixed, parent right_middle_pip_jointbody, child right_middle_ip_sensor_6, origin xyz=-0.0 -0.0 -0.0 rpy=0.0 0.0 0.0
- added joint right_middle_pip_sensor_7_joint: type fixed, parent right_middle_pip_jointbody, child right_middle_ip_sensor_7, origin xyz=-0.0 -0.0 -0.0 rpy=0.0 0.0 0.0
- added joint right_middle_pip_sensor_8_joint: type fixed, parent right_middle_pip_jointbody, child right_middle_ip_sensor_8, origin xyz=-0.0 -0.0 -0.0 rpy=0.0 0.0 0.0
- added joint right_middle_pip_sensor_9_joint: type fixed, parent right_middle_pip_jointbody, child right_middle_ip_sensor_9, origin xyz=-0.0 -0.0 -0.0 rpy=0.0 0.0 0.0
