Commit message: added thumb in model && updated urdf

File: models/urdf/orcahand.urdf (robot description, URDF)
Before this commit: robot orcahand, 57 links, 56 joints
Links:
- added link right_thumb_dp_sensor_10, mass 1e-8; collision mesh filename=package://orcahand_description/assets/urdf/collision/thumb_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 scale=1 1 1; visual mesh filename=package://orcahand_description/assets/urdf/visual/thumb_dp_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 scale=1 1 1
- added link right_thumb_dp_sensor_11, mass 1e-8; collision mesh filename=package://orcahand_description/assets/urdf/collision/thumb_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 scale=1 1 1; visual mesh filename=package://orcahand_description/assets/urdf/visual/thumb_dp_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 scale=1 1 1
- added link right_thumb_dp_sensor_12, mass 1e-8; collision mesh filename=package://orcahand_description/assets/urdf/collision/thumb_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 scale=1 1 1; visual mesh filename=package://orcahand_description/assets/urdf/visual/thumb_dp_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 scale=1 1 1
- added link right_thumb_dp_sensor_13, mass 1e-8; collision mesh filename=package://orcahand_description/assets/urdf/collision/thumb_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 scale=1 1 1; visual mesh filename=package://orcahand_description/assets/urdf/visual/thumb_dp_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 scale=1 1 1
- added link right_thumb_dp_sensor_2, mass 1e-8; collision mesh filename=package://orcahand_description/assets/urdf/collision/thumb_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 scale=1 1 1; visual mesh filename=package://orcahand_description/assets/urdf/visual/thumb_dp_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 scale=1 1 1
- added link right_thumb_dp_sensor_3, mass 1e-8; collision mesh filename=package://orcahand_description/assets/urdf/collision/thumb_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 scale=1 1 1; visual mesh filename=package://orcahand_description/assets/urdf/visual/thumb_dp_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 scale=1 1 1
- added link right_thumb_dp_sensor_4, mass 1e-8; collision mesh filename=package://orcahand_description/assets/urdf/collision/thumb_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 scale=1 1 1; visual mesh filename=package://orcahand_description/assets/urdf/visual/thumb_dp_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 scale=1 1 1
- added link right_thumb_dp_sensor_5, mass 1e-8; collision mesh filename=package://orcahand_description/assets/urdf/collision/thumb_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 scale=1 1 1; visual mesh filename=package://orcahand_description/assets/urdf/visual/thumb_dp_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 scale=1 1 1
- added link right_thumb_dp_sensor_6, mass 1e-8; collision mesh filename=package://orcahand_description/assets/urdf/collision/thumb_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 scale=1 1 1; visual mesh filename=package://orcahand_description/assets/urdf/visual/thumb_dp_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 scale=1 1 1
- added link right_thumb_dp_sensor_7, mass 1e-8; collision mesh filename=package://orcahand_description/assets/urdf/collision/thumb_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 scale=1 1 1; visual mesh filename=package://orcahand_description/assets/urdf/visual/thumb_dp_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 scale=1 1 1
- added link right_thumb_dp_sensor_8, mass 1e-8; collision mesh filename=package://orcahand_description/assets/urdf/collision/thumb_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 scale=1 1 1; visual mesh filename=package://orcahand_description/assets/urdf/visual/thumb_dp_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 scale=1 1 1
- added link right_thumb_dp_sensor_9, mass 1e-8; collision mesh filename=package://orcahand_description/assets/urdf/collision/thumb_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 scale=1 1 1; visual mesh filename=package://orcahand_description/assets/urdf/visual/thumb_dp_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 scale=1 1 1
Joints:
- added joint right_thumb_dip_sensor_10_joint: type fixed, parent right_thumb_dip_jointbody, child right_thumb_dp_sensor_10, origin xyz=-0.0 -0.0 -0.0 rpy=0.0 0.0 0.0
- added joint right_thumb_dip_sensor_11_joint: type fixed, parent right_thumb_dip_jointbody, child right_thumb_dp_sensor_11, origin xyz=-0.0 -0.0 -0.0 rpy=0.0 0.0 0.0
- added joint right_thumb_dip_sensor_12_joint: type fixed, parent right_thumb_dip_jointbody, child right_thumb_dp_sensor_12, origin xyz=-0.0 -0.0 -0.0 rpy=0.0 0.0 0.0
- added joint right_thumb_dip_sensor_13_joint: type fixed, parent right_thumb_dip_jointbody, child right_thumb_dp_sensor_13, origin xyz=-0.0 -0.0 -0.0 rpy=0.0 0.0 0.0
- added joint right_thumb_dip_sensor_2_joint: type fixed, parent right_thumb_dip_jointbody, child right_thumb_dp_sensor_2, origin xyz=-0.0 -0.0 -0.0 rpy=0.0 0.0 0.0
- added joint right_thumb_dip_sensor_3_joint: type fixed, parent right_thumb_dip_jointbody, child right_thumb_dp_sensor_3, origin xyz=-0.0 -0.0 -0.0 rpy=0.0 0.0 0.0
- added joint right_thumb_dip_sensor_4_joint: type fixed, parent right_thumb_dip_jointbody, child right_thumb_dp_sensor_4, origin xyz=-0.0 -0.0 -0.0 rpy=0.0 0.0 0.0
- added joint right_thumb_dip_sensor_5_joint: type fixed, parent right_thumb_dip_jointbody, child right_thumb_dp_sensor_5, origin xyz=-0.0 -0.0 -0.0 rpy=0.0 0.0 0.0
- added joint right_thumb_dip_sensor_6_joint: type fixed, parent right_thumb_dip_jointbody, child right_thumb_dp_sensor_6, origin xyz=-0.0 -0.0 -0.0 rpy=0.0 0.0 0.0
- added joint right_thumb_dip_sensor_7_joint: type fixed, parent right_thumb_dip_jointbody, child right_thumb_dp_sensor_7, origin xyz=-0.0 -0.0 -0.0 rpy=0.0 0.0 0.0
- added joint right_thumb_dip_sensor_8_joint: type fixed, parent right_thumb_dip_jointbody, child right_thumb_dp_sensor_8, origin xyz=-0.0 -0.0 -0.0 rpy=0.0 0.0 0.0
- added joint right_thumb_dip_sensor_9_joint: type fixed, parent right_thumb_dip_jointbody, child right_thumb_dp_sensor_9, origin xyz=-0.0 -0.0 -0.0 rpy=0.0 0.0 0.0

File: models/urdf/orcahand.urdf.xacro (robot description, xacro)
@@ -412,5 +412,5 @@
          <inertia ixx="1e-8" iyy="1e-8" izz="1e-8" ixy="0.0" ixz="0.0" iyz="0.0"/>
       </inertial>
-      <visual name="${prefix}visual_thumb_dp_skin_mesh_surface_1">
+      <visual name="${prefix}visual_thumb_dp_skin_mesh_surface">
          <origin xyz="${s * 0.002793435568551968} -6.14386555467744e-07 0.016601042013200628" rpy="3.141592653589793 ${s * -0.40239793279263236} 0.0"/>
          <geometry>
@@ -419,7 +419,7 @@
             />
          </geometry>
-         <material name="red"/>
-      </visual>
-      <collision name="${prefix}collision_thumb_dp_skin_mesh_surface_1">
+         <material name="yellow"/>
+      </visual>
+      <collision name="${prefix}collision_thumb_dp_skin_mesh_surface">
          <origin xyz="${s * 0.002785448336058668} -6.944475247259374e-06 0.016557497442018437" rpy="3.141592653589793 ${s * -0.3963953079219906} 0.0"/>
          <geometry>
@@ -428,5 +428,305 @@
             />
          </geometry>
-         <material name="green"/>
+         <material name="yellow"/>
+      </collision>
+   </link>
+   <link name="${prefix}thumb_dp_sensor_2">
+      <inertial>
+         <origin xyz="0.00233 1e-05 0.01133" rpy="0.00075 0.08211000000000013 0.00013000000000000002"/>
+         <mass value="1e-8"/>
+         <inertia ixx="1e-8" iyy="1e-8" izz="1e-8" ixy="0.0" ixz="0.0" iyz="0.0"/>
+      </inertial>
+      <visual name="${prefix}visual_thumb_dp_skin_mesh_surface">
+         <origin xyz="${s * 0.002793435568551968} -6.14386555467744e-07 0.016601042013200628" rpy="3.141592653589793 ${s * -0.40239793279263236} 0.0"/>
+         <geometry>
+            <mesh filename="${rospackage_path}/visual/thumb_dp_skin_mesh_surface_2.stl"
+            scale="${'-1 1 1' if chirality == 'left' else '1 1 1'}"
+            />
+         </geometry>
+         <material name="magenta"/>
+      </visual>
+      <collision name="${prefix}collision_thumb_dp_skin_mesh_surface">
+         <origin xyz="${s * 0.002785448336058668} -6.944475247259374e-06 0.016557497442018437" rpy="3.141592653589793 ${s * -0.3963953079219906} 0.0"/>
+         <geometry>
+            <mesh filename="${rospackage_path}/collision/thumb_dp_skin_mesh_surface_2.stl"
+            scale="${'-1 1 1' if chirality == 'left' else '1 1 1'}"
+            />
+         </geometry>
+         <material name="magenta"/>
+      </collision>
+   </link>
+   <link name="${prefix}thumb_dp_sensor_3">
+      <inertial>
+         <origin xyz="0.00233 1e-05 0.01133" rpy="0.00075 0.08211000000000013 0.00013000000000000002"/>
+         <mass value="1e-8"/>
+         <inertia ixx="1e-8" iyy="1e-8" izz="1e-8" ixy="0.0" ixz="0.0" iyz="0.0"/>
+      </inertial>
+      <visual name="${prefix}visual_thumb_dp_skin_mesh_surface">
+         <origin xyz="${s * 0.002793435568551968} -6.14386555467744e-07 0.016601042013200628" rpy="3.141592653589793 ${s * -0.40239793279263236} 0.0"/>
+         <geometry>
+            <mesh filename="${rospackage_path}/visual/thumb_dp_skin_mesh_surface_3.stl"
+            scale="${'-1 1 1' if chirality == 'left' else '1 1 1'}"
+            />
+         </geometry>
+         <material name="cyan"/>
+      </visual>
+      <collision name="${prefix}collision_thumb_dp_skin_mesh_surface">
+         <origin xyz="${s * 0.002785448336058668} -6.944475247259374e-06 0.016557497442018437" rpy="3.141592653589793 ${s * -0.3963953079219906} 0.0"/>
+         <geometry>
+            <mesh filename="${rospackage_path}/collision/thumb_dp_skin_mesh_surface_3.stl"
+            scale="${'-1 1 1' if chirality == 'left' else '1 1 1'}"
+            />
+         </geometry>
+         <material name="cyan"/>
+      </collision>
+   </link>
+   <link name="${prefix}thumb_dp_sensor_4">
+      <inertial>
+         <origin xyz="0.00233 1e-05 0.01133" rpy="0.00075 0.08211000000000013 0.00013000000000000002"/>
+         <mass value="1e-8"/>
+         <inertia ixx="1e-8" iyy="1e-8" izz="1e-8" ixy="0.0" ixz="0.0" iyz="0.0"/>
+      </inertial>
+      <visual name="${prefix}visual_thumb_dp_skin_mesh_surface">
+         <origin xyz="${s * 0.002793435568551968} -6.14386555467744e-07 0.016601042013200628" rpy="3.141592653589793 ${s * -0.40239793279263236} 0.0"/>
+         <geometry>
+            <mesh filename="${rospackage_path}/visual/thumb_dp_skin_mesh_surface_4.stl"
+            scale="${'-1 1 1' if chirality == 'left' else '1 1 1'}"
+            />
+         </geometry>
+         <material name="blue"/>
+      </visual>
+      <collision name="${prefix}collision_thumb_dp_skin_mesh_surface">
+         <origin xyz="${s * 0.002785448336058668} -6.944475247259374e-06 0.016557497442018437" rpy="3.141592653589793 ${s * -0.3963953079219906} 0.0"/>
+         <geometry>
+            <mesh filename="${rospackage_path}/collision/thumb_dp_skin_mesh_surface_4.stl"
+            scale="${'-1 1 1' if chirality == 'left' else '1 1 1'}"
+            />
+         </geometry>
+         <material name="blue"/>
+      </collision>
+   </link>
+   <link name="${prefix}thumb_dp_sensor_5">
+      <inertial>
+         <origin xyz="0.00233 1e-05 0.01133" rpy="0.00075 0.08211000000000013 0.00013000000000000002"/>
+         <mass value="1e-8"/>
+         <inertia ixx="1e-8" iyy="1e-8" izz="1e-8" ixy="0.0" ixz="0.0" iyz="0.0"/>
+      </inertial>
+      <visual name="${prefix}visual_thumb_dp_skin_mesh_surface">
+         <origin xyz="${s * 0.002793435568551968} -6.14386555467744e-07 0.016601042013200628" rpy="3.141592653589793 ${s * -0.40239793279263236} 0.0"/>
+         <geometry>
+            <mesh filename="${rospackage_path}/visual/thumb_dp_skin_mesh_surface_5.stl"
+            scale="${'-1 1 1' if chirality == 'left' else '1 1 1'}"
+            />
+         </geometry>
+         <material name="yellow"/>
+      </visual>
+      <collision name="${prefix}collision_thumb_dp_skin_mesh_surface">
+         <origin xyz="${s * 0.002785448336058668} -6.944475247259374e-06 0.016557497442018437" rpy="3.141592653589793 ${s * -0.3963953079219906} 0.0"/>
+         <geometry>
+            <mesh filename="${rospackage_path}/collision/thumb_dp_skin_mesh_surface_5.stl"
+            scale="${'-1 1 1' if chirality == 'left' else '1 1 1'}"
+            />
+         </geometry>
+         <material name="yellow"/>
+      </collision>
+   </link>
+   <link name="${prefix}thumb_dp_sensor_6">
+      <inertial>
+         <origin xyz="0.00233 1e-05 0.01133" rpy="0.00075 0.08211000000000013 0.00013000000000000002"/>
+         <mass value="1e-8"/>
+         <inertia ixx="1e-8" iyy="1e-8" izz="1e-8" ixy="0.0" ixz="0.0" iyz="0.0"/>
+      </inertial>
+      <visual name="${prefix}visual_thumb_dp_skin_mesh_surface">
+         <origin xyz="${s * 0.002793435568551968} -6.14386555467744e-07 0.016601042013200628" rpy="3.141592653589793 ${s * -0.40239793279263236} 0.0"/>
+         <geometry>
+            <mesh filename="${rospackage_path}/visual/thumb_dp_skin_mesh_surface_6.stl"
+            scale="${'-1 1 1' if chirality == 'left' else '1 1 1'}"
+            />
+         </geometry>
+         <material name="magenta"/>
+      </visual>
+      <collision name="${prefix}collision_thumb_dp_skin_mesh_surface">
+         <origin xyz="${s * 0.002785448336058668} -6.944475247259374e-06 0.016557497442018437" rpy="3.141592653589793 ${s * -0.3963953079219906} 0.0"/>
+         <geometry>
+            <mesh filename="${rospackage_path}/collision/thumb_dp_skin_mesh_surface_6.stl"
+            scale="${'-1 1 1' if chirality == 'left' else '1 1 1'}"
+            />
+         </geometry>
+         <material name="magenta"/>
+      </collision>
+   </link>
+   <link name="${prefix}thumb_dp_sensor_7">
+      <inertial>
+         <origin xyz="0.00233 1e-05 0.01133" rpy="0.00075 0.08211000000000013 0.00013000000000000002"/>
+         <mass value="1e-8"/>
+         <inertia ixx="1e-8" iyy="1e-8" izz="1e-8" ixy="0.0" ixz="0.0" iyz="0.0"/>
+      </inertial>
+      <visual name="${prefix}visual_thumb_dp_skin_mesh_surface">
+         <origin xyz="${s * 0.002793435568551968} -6.14386555467744e-07 0.016601042013200628" rpy="3.141592653589793 ${s * -0.40239793279263236} 0.0"/>
+         <geometry>
+            <mesh filename="${rospackage_path}/visual/thumb_dp_skin_mesh_surface_7.stl"
+            scale="${'-1 1 1' if chirality == 'left' else '1 1 1'}"
+            />
+         </geometry>
+         <material name="cyan"/>
+      </visual>
+      <collision name="${prefix}collision_thumb_dp_skin_mesh_surface">
+         <origin xyz="${s * 0.002785448336058668} -6.944475247259374e-06 0.016557497442018437" rpy="3.141592653589793 ${s * -0.3963953079219906} 0.0"/>
+         <geometry>
+            <mesh filename="${rospackage_path}/collision/thumb_dp_skin_mesh_surface_7.stl"
+            scale="${'-1 1 1' if chirality == 'left' else '1 1 1'}"
+            />
+         </geometry>
+         <material name="cyan"/>
+      </collision>
+   </link>
+   <link name="${prefix}thumb_dp_sensor_8">
+      <inertial>
+         <origin xyz="0.00233 1e-05 0.01133" rpy="0.00075 0.08211000000000013 0.00013000000000000002"/>
+         <mass value="1e-8"/>
+         <inertia ixx="1e-8" iyy="1e-8" izz="1e-8" ixy="0.0" ixz="0.0" iyz="0.0"/>
+      </inertial>
+      <visual name="${prefix}visual_thumb_dp_skin_mesh_surface">
+         <origin xyz="${s * 0.002793435568551968} -6.14386555467744e-07 0.016601042013200628" rpy="3.141592653589793 ${s * -0.40239793279263236} 0.0"/>
+         <geometry>
+            <mesh filename="${rospackage_path}/visual/thumb_dp_skin_mesh_surface_8.stl"
+            scale="${'-1 1 1' if chirality == 'left' else '1 1 1'}"
+            />
+         </geometry>
+         <material name="blue"/>
+      </visual>
+      <collision name="${prefix}collision_thumb_dp_skin_mesh_surface">
+         <origin xyz="${s * 0.002785448336058668} -6.944475247259374e-06 0.016557497442018437" rpy="3.141592653589793 ${s * -0.3963953079219906} 0.0"/>
+         <geometry>
+            <mesh filename="${rospackage_path}/collision/thumb_dp_skin_mesh_surface_8.stl"
+            scale="${'-1 1 1' if chirality == 'left' else '1 1 1'}"
+            />
+         </geometry>
+         <material name="blue"/>
+      </collision>
+   </link>
+   <link name="${prefix}thumb_dp_sensor_9">
+      <inertial>
+         <origin xyz="0.00233 1e-05 0.01133" rpy="0.00075 0.08211000000000013 0.00013000000000000002"/>
+         <mass value="1e-8"/>
+         <inertia ixx="1e-8" iyy="1e-8" izz="1e-8" ixy="0.0" ixz="0.0" iyz="0.0"/>
+      </inertial>
+      <visual name="${prefix}visual_thumb_dp_skin_mesh_surface">
+         <origin xyz="${s * 0.002793435568551968} -6.14386555467744e-07 0.016601042013200628" rpy="3.141592653589793 ${s * -0.40239793279263236} 0.0"/>
+         <geometry>
+            <mesh filename="${rospackage_path}/visual/thumb_dp_skin_mesh_surface_9.stl"
+            scale="${'-1 1 1' if chirality == 'left' else '1 1 1'}"
+            />
+         </geometry>
+         <material name="yellow"/>
+      </visual>
+      <collision name="${prefix}collision_thumb_dp_skin_mesh_surface">
+         <origin xyz="${s * 0.002785448336058668} -6.944475247259374e-06 0.016557497442018437" rpy="3.141592653589793 ${s * -0.3963953079219906} 0.0"/>
+         <geometry>
+            <mesh filename="${rospackage_path}/collision/thumb_dp_skin_mesh_surface_9.stl"
+            scale="${'-1 1 1' if chirality == 'left' else '1 1 1'}"
+            />
+         </geometry>
+         <material name="yellow"/>
+      </collision>
+   </link>
+   <link name="${prefix}thumb_dp_sensor_10">
+      <inertial>
+         <origin xyz="0.00233 1e-05 0.01133" rpy="0.00075 0.08211000000000013 0.00013000000000000002"/>
+         <mass value="1e-8"/>
+         <inertia ixx="1e-8" iyy="1e-8" izz="1e-8" ixy="0.0" ixz="0.0" iyz="0.0"/>
+      </inertial>
+      <visual name="${prefix}visual_thumb_dp_skin_mesh_surface">
+         <origin xyz="${s * 0.002793435568551968} -6.14386555467744e-07 0.016601042013200628" rpy="3.141592653589793 ${s * -0.40239793279263236} 0.0"/>
+         <geometry>
+            <mesh filename="${rospackage_path}/visual/thumb_dp_skin_mesh_surface_10.stl"
+            scale="${'-1 1 1' if chirality == 'left' else '1 1 1'}"
+            />
+         </geometry>
+         <material name="cyan"/>
+      </visual>
+      <collision name="${prefix}collision_thumb_dp_skin_mesh_surface">
+         <origin xyz="${s * 0.002785448336058668} -6.944475247259374e-06 0.016557497442018437" rpy="3.141592653589793 ${s * -0.3963953079219906} 0.0"/>
+         <geometry>
+            <mesh filename="${rospackage_path}/collision/thumb_dp_skin_mesh_surface_10.stl"
+            scale="${'-1 1 1' if chirality == 'left' else '1 1 1'}"
+            />
+         </geometry>
+         <material name="cyan"/>
+      </collision>
+   </link>
+   <link name="${prefix}thumb_dp_sensor_11">
+      <inertial>
+         <origin xyz="0.00233 1e-05 0.01133" rpy="0.00075 0.08211000000000013 0.00013000000000000002"/>
+         <mass value="1e-8"/>
+         <inertia ixx="1e-8" iyy="1e-8" izz="1e-8" ixy="0.0" ixz="0.0" iyz="0.0"/>
+      </inertial>
+      <visual name="${prefix}visual_thumb_dp_skin_mesh_surface">
+         <origin xyz="${s * 0.002793435568551968} -6.14386555467744e-07 0.016601042013200628" rpy="3.141592653589793 ${s * -0.40239793279263236} 0.0"/>
+         <geometry>
+            <mesh filename="${rospackage_path}/visual/thumb_dp_skin_mesh_surface_11.stl"
+            scale="${'-1 1 1' if chirality == 'left' else '1 1 1'}"
+            />
+         </geometry>
+         <material name="magenta"/>
+      </visual>
+      <collision name="${prefix}collision_thumb_dp_skin_mesh_surface">
+         <origin xyz="${s * 0.002785448336058668} -6.944475247259374e-06 0.016557497442018437" rpy="3.141592653589793 ${s * -0.3963953079219906} 0.0"/>
+         <geometry>
+            <mesh filename="${rospackage_path}/collision/thumb_dp_skin_mesh_surface_11.stl"
+            scale="${'-1 1 1' if chirality == 'left' else '1 1 1'}"
+            />
+         </geometry>
+         <material name="magenta"/>
+      </collision>
+   </link>
+   <link name="${prefix}thumb_dp_sensor_12">
+      <inertial>
+         <origin xyz="0.00233 1e-05 0.01133" rpy="0.00075 0.08211000000000013 0.00013000000000000002"/>
+         <mass value="1e-8"/>
+         <inertia ixx="1e-8" iyy="1e-8" izz="1e-8" ixy="0.0" ixz="0.0" iyz="0.0"/>
+      </inertial>
+      <visual name="${prefix}visual_thumb_dp_skin_mesh_surface">
+         <origin xyz="${s * 0.002793435568551968} -6.14386555467744e-07 0.016601042013200628" rpy="3.141592653589793 ${s * -0.40239793279263236} 0.0"/>
+         <geometry>
+            <mesh filename="${rospackage_path}/visual/thumb_dp_skin_mesh_surface_12.stl"
+            scale="${'-1 1 1' if chirality == 'left' else '1 1 1'}"
+            />
+         </geometry>
+         <material name="blue"/>
+      </visual>
+      <collision name="${prefix}collision_thumb_dp_skin_mesh_surface">
+         <origin xyz="${s * 0.002785448336058668} -6.944475247259374e-06 0.016557497442018437" rpy="3.141592653589793 ${s * -0.3963953079219906} 0.0"/>
+         <geometry>
+            <mesh filename="${rospackage_path}/collision/thumb_dp_skin_mesh_surface_12.stl"
+            scale="${'-1 1 1' if chirality == 'left' else '1 1 1'}"
+            />
+         </geometry>
+         <material name="blue"/>
+      </collision>
+   </link>
+   <link name="${prefix}thumb_dp_sensor_13">
+      <inertial>
+         <origin xyz="0.00233 1e-05 0.01133" rpy="0.00075 0.08211000000000013 0.00013000000000000002"/>
+         <mass value="1e-8"/>
+         <inertia ixx="1e-8" iyy="1e-8" izz="1e-8" ixy="0.0" ixz="0.0" iyz="0.0"/>
+      </inertial>
+      <visual name="${prefix}visual_thumb_dp_skin_mesh_surface">
+         <origin xyz="${s * 0.002793435568551968} -6.14386555467744e-07 0.016601042013200628" rpy="3.141592653589793 ${s * -0.40239793279263236} 0.0"/>
+         <geometry>
+            <mesh filename="${rospackage_path}/visual/thumb_dp_skin_mesh_surface_13.stl"
+            scale="${'-1 1 1' if chirality == 'left' else '1 1 1'}"
+            />
+         </geometry>
+         <material name="yellow"/>
+      </visual>
+      <collision name="${prefix}collision_thumb_dp_skin_mesh_surface">
+         <origin xyz="${s * 0.002785448336058668} -6.944475247259374e-06 0.016557497442018437" rpy="3.141592653589793 ${s * -0.3963953079219906} 0.0"/>
+         <geometry>
+            <mesh filename="${rospackage_path}/collision/thumb_dp_skin_mesh_surface_13.stl"
+            scale="${'-1 1 1' if chirality == 'left' else '1 1 1'}"
+            />
+         </geometry>
+         <material name="yellow"/>
       </collision>
    </link>
@@ -455,5 +755,5 @@
       <origin xyz="-0.0 -0.0 -0.0" rpy="0.0 0.0 0.0"/>
    </joint>
-   <!-- <joint type="fixed" name="${prefix}thumb_dip_sensor_2_joint">
+   <joint type="fixed" name="${prefix}thumb_dip_sensor_2_joint">
       <parent link="${prefix}thumb_dip_jointbody"/>
       <child link="${prefix}thumb_dp_sensor_2"/>
@@ -515,5 +815,5 @@
       <origin xyz="-0.0 -0.0 -0.0" rpy="0.0 0.0 0.0"/>
    </joint>
-   <joint type="fixed" name="${prefix}thumb_dip_sensor_14_joint">
+   <!-- <joint type="fixed" name="${prefix}thumb_dip_sensor_14_joint">
       <parent link="${prefix}thumb_dip_jointbody"/>
       <child link="${prefix}thumb_dp_sensor_14"/>
